File: Lcd16x2_Backpack.brd (EAGLE design)
At the start: 22 parts, among them IC1 REG1117, IC3 74HCT595N

Commit message: Production 1
Parts:
- removed U$3: HEADER-4PIN, GlennTamayoEagle:HEADER-4PIN
- removed U$4: HEADER-2PINA, GlennTamayoEagle:HEADER-2PIN
- added U$16, U$17: CAPACITOR-0.2-CER1206, GlennTamayoEagle:1206
- moved U$12 69.2 mm to (47.9, 12.1), flipped to the bottom
- moved U$13 62.6 mm to (41.9, 6.67), flipped to the bottom, turned to 90 degrees
- moved IC1 62.2 mm to (48.9, 7.30), flipped to the bottom, turned to 90 degrees
- moved U$10 59.4 mm to (32.4, 28.9)
- moved U$8 44.7 mm to (30.8, 23.2), flipped to the bottom, turned to 180 degrees
- moved U$7 40.9 mm to (30.8, 20.3), flipped to the bottom, turned to 180 degrees
- moved U$9 38.7 mm to (5.40, 24.1), turned to 270 degrees
- moved U$11 33.7 mm to (6.03, 4.76), turned to 90 degrees
- moved U$5 22.6 mm to (6.03, 14.9)
- moved U$6 17.2 mm to (6.03, 12.1), flipped to the bottom
- moved U$1 16.6 mm to (6.03, 9.21), flipped to the bottom, turned to 180 degrees
- moved SJR1 5.17 mm to (19.1, 15.9)
Connections:
- removed net 595CLOCK: SJR1.5
- net 3V3: now also U$16.2, U$17.2
- net 595RCK: now also SJR1.5; no longer SJR1.13, U$3.3
- net 595SCK: now also SJR1.4; no longer U$3.2
- net 595SER: no longer U$3.4
- net GND: now also U$16.1, U$17.1; no longer U$4.1, U$4.2
- net RX: now also U$9.3; no longer U$9.2
- net TX: now also U$9.2; no longer U$9.3
- net VCC: no longer U$3.1
Routing:
- net GND: track 29.4 -> 214.6 mm
- net 3V3: track 0.00 -> 80.8 mm, vias 0 -> 3
- net 595SER: track 5.05 -> 54.9 mm
- net 595RCK: track 4.26 -> 47.5 mm
- net 595SCK: track 4.26 -> 44.7 mm
- net N$5: track 0.00 -> 29.5 mm
- net N$1: track 0.00 -> 20.5 mm
- net TX: track 0.00 -> 6.60 mm
- net RX: track 0.00 -> 6.38 mm
- net N$3: track 0.00 -> 3.51 mm
- net N$4: track 0.00 -> 3.33 mm
- net N$2: track 0.00 -> 3.18 mm
- net VCC: track 107.6 -> 109.8 mm, vias 2 -> 1
Other:
- board text added: "gt"
- board text removed: "gtamayo"
