File: Lcd16x2_Backpack.sch (EAGLE design)
At the start: 22 parts, among them IC1 REG1117, IC3 74HCT595N

Commit message: Update Lcd16x2_Backpack.sch
Parts:
- removed U$3: HEADER-4PIN, GlennTamayoEagle:HEADER-4PIN
- removed U$4: HEADER-2PINA, GlennTamayoEagle:HEADER-2PINA
- added U$16, U$17: CAPACITOR-0.2-CER1206, GlennTamayoEagle:CAPACITOR-0.2-CER1206
Connections:
- removed net 595CLOCK: SJR1.GPIO14
- net 3V3: now also U$16.2, U$17.2
- net 595RCK: now also SJR1.GPIO14; no longer SJR1.GPIO4, U$3.3
- net 595SCK: now also SJR1.GPIO16; no longer U$3.2
- net 595SER: no longer U$3.4
- net GND: now also U$16.1, U$17.1; no longer U$4.2, U$4.3
- net RX: now also U$9.3; no longer U$9.2
- net TX: now also U$9.2; no longer U$9.3
- net VCC: no longer U$3.1
